File: head/main/head-main.kicad_sch (KiCad schematic)
At the start: 54 parts, among them J1 conn_head_b, U1 CV1800B, U2 AR0237CS, U3 GTA2718B-3HA, U4 W25Q128JVP, Y1 25M

Commit message: update communication pinout
Parts:
- J1: value conn_head_b -> conn_head_comms
Connections:
- net +1V8: now also J1.18 (Pin_18); no longer J1.6 (Pin_6)
- net U3RX: now also J1.12 (Pin_12); no longer J1.14 (Pin_14)
- net U3TX: now also J1.14 (Pin_14); no longer J1.12 (Pin_12)
- net USB_DM: now also J1.6 (Pin_6); no longer J1.8 (Pin_8)
- net USB_DP: now also J1.8 (Pin_8); no longer J1.10 (Pin_10)
- net U3CTS renamed UDIR
- net U3RTS renamed LED
- net LED: now also J1.10 (Pin_10); no longer J1.18 (Pin_18)

Commit message: finishing touches
Parts:
- C1, C11, C15, C19, C2, C22, C24, C27, C29, C3, C31, C4, C41, C43, C8, C9: value 0.1u -> 100n; LCSC (none) -> *
- C10, C14, C17, C20, C21, C23, C25, C26, C28, C30, C32, C33, C34, C35, C36, C37, C39, C40, C42, C5, C6, C7, R1, R3, R4, R5: LCSC (none) -> *
- H1, H2, H3, H4, H5, H6, U1: LCSC (none) -> -
