File: head/main/power.kicad_sch (KiCad schematic)
At the start: 23 parts, among them U5 RP509x, U6 RP509x, U7 RP114x, U8 LP3982S, U9 NCP136

Commit message: update title
Other:
- title: HW1 / Head / Main -> HW1 / Head / Main - Power
Changed lines of the file:
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@@
 	(paper "A5")
 	(title_block
-		(title "HW1 / Head / Main")
+		(title "HW1 / Head / Main - Power")
 		(date "2025-10-07")
 		(rev "1")

Commit message: update communication pinout
Other:
- title: HW1 / Head / Main - Power -> HW1 / Head / Main
Changed lines of the file:
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@@
 	(paper "A5")
 	(title_block
-		(title "HW1 / Head / Main - Power")
+		(title "HW1 / Head / Main")
 		(date "2025-10-07")
 		(rev "1")
 		(company "team noon")
+		(comment 1 "NanoID: AZq9ZVGu")
 		(comment 3 "github.com/team-noon/hw1")
 		(comment 4 "Drawn By: Sam")

Commit message: finishing touches
Parts:
- C50, C51, C52, C53, C54, C55, C57, C58, C60, C61, C65: LCSC (none) -> *
- C63: value 4.7u (Cin) -> 4.7u; LCSC (none) -> *
- R10: value 440k -> 44k; LCSC (none) -> *
- R6: value 220k -> 44k; LCSC (none) -> *
- R7: value 220k -> 22k; LCSC (none) -> *
- R9: value 110k -> 22k; LCSC (none) -> *
Changed lines of the file:
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@@
 		(rev "1")
 		(company "team noon")
-		(comment 1 "NanoID: AZq9ZVGu")
+		(comment 1 "NanoID: NAFCDP")
 		(comment 3 "github.com/team-noon/hw1")
 		(comment 4 "Drawn By: Sam")
@@
 			)
 		)
+		(property "LCSC" "*"
+			(at 78.74 95.25 0)
+			(hide yes)
+			(show_name no)
+			(do_not_autoplace no)
+			(effects
+				(font
+					(size 1.27 1.27)
+				)
+			)
+		)
 		(pin "2"
 		)
@@
 			)
 		)
+		(property "LCSC" "*"
+			(at 78.74 77.47 0)
+			(hide yes)
+			(show_name no)
+			(do_not_autoplace no)
+			(effects
+				(font
+					(size 1.27 1.27)
+				)
+			)
+		)
 		(pin "2"
 		)
@@
 			)
 		)
+		(property "LCSC" "*"
+			(at 78.74 33.02 0)
+			(hide yes)
+			(show_name no)
+			(do_not_autoplace no)
+			(effects
+				(font
+					(size 1.27 1.27)
+				)
+			)
+		)
 		(pin "1"
 		)
@@
 			)
 		)
-		(property "Value" "110k"
+		(property "Value" "22k"
 			(at 71.12 30.48 90)
 			(hide yes)
@@
 			)
 		)
+		(property "LCSC" "*"
+			(at 71.12 33.02 90)
+			(hide yes)
+			(show_name no)
+			(do_not_autoplace no)
+			(effects
+				(font
+					(size 1.27 1.27)
+				)
+			)
+		)
 		(pin "1"
 		)
@@
 			)
 		)
-		(property "Value" "220k"
+		(property "Value" "22k"
 			(at 63.5 57.15 90)
 			(hide yes)
@@
 			)
 		)
+		(property "LCSC" "*"
+			(at 63.5 59.69 90)
+			(hide yes)
+			(show_name no)
+			(do_not_autoplace no)
+			(effects
+				(font
+					(size 1.27 1.27)
+				)
+			)
+		)
 		(pin "1"
 		)
@@
 			)
 		)
+		(property "LCSC" "*"
+			(at 34.29 55.88 0)
+			(hide yes)
+			(show_name no)
+			(do_not_autoplace no)
+			(effects
+				(font
+					(size 1.27 1.27)
+				)
+			)
+		)
 		(pin "1"
 		)
@@
 			)
 		)
+		(property "LCSC" "*"
+			(at 34.29 77.47 0)
+			(hide yes)
+			(show_name no)
+			(do_not_autoplace no)
+			(effects
+				(font
+					(size 1.27 1.27)
+				)
+			)
+		)
 		(pin "2"
 		)
@@
 			)
 		)
-		(property "Value" "220k"
+		(property "Value" "44k"
 			(at 63.5 34.29 90)
 			(hide yes)
@@
 			)
 		)
+		(property "LCSC" "*"
+			(at 63.5 36.83 90)
+			(hide yes)
+			(show_name no)
+			(do_not_autoplace no)
+			(effects
+				(font
+					(size 1.27 1.27)
+				)
+			)
+		)
 		(pin "1"
 		)
@@
 			)
 		)
-		(property "Value" "440k"
+		(property "Value" "44k"
 			(at 71.12 53.34 90)
 			(hide yes)
@@
 			)
 		)
+		(property "LCSC" "*"
+			(at 71.12 55.88 90)
+			(hide yes)
+			(show_name no)
+			(do_not_autoplace no)
+			(effects
+				(font
+					(size 1.27 1.27)
+				)
+			)
+		)
 		(pin "1"
 		)
@@
 			)
 		)
+		(property "LCSC" "*"
+			(at 78.74 55.88 0)
+			(hide yes)
+			(show_name no)
+			(do_not_autoplace no)
+			(effects
+				(font
+					(size 1.27 1.27)
+				)
+			)
+		)
 		(pin "1"
 		)
@@
 			)
 		)
+		(property "LCSC" "*"
+			(at 34.29 95.25 0)
+			(hide yes)
+			(show_name no)
+			(do_not_autoplace no)
+			(effects
+				(font
+					(size 1.27 1.27)
+				)
+			)
+		)
 		(pin "2"
 		)
@@
 			)
 		)
+		(property "LCSC" "*"
+			(at 120.65 55.88 0)
+			(hide yes)
+			(show_name no)
+			(do_not_autoplace no)
+			(effects
+				(font
+					(size 1.27 1.27)
+				)
+			)
+		)
 		(pin "2"
 		)
@@
 			)
 		)
+		(property "LCSC" "*"
+			(at 34.29 33.02 0)
+			(hide yes)
+			(show_name no)
+			(do_not_autoplace no)
+			(effects
+				(font
+					(size 1.27 1.27)
+				)
+			)
+		)
 		(pin "1"
 		)
@@
 			)
 		)
-		(property "Value" "4.7u (Cin)"
+		(property "Value" "4.7u"
 			(at 99.06 57.1499 0)
 			(hide yes)
@@
 			)
 		)
+		(property "LCSC" "*"
+			(at 95.25 55.88 0)
+			(hide yes)
+			(show_name no)
+			(do_not_autoplace no)
+			(effects
+				(font
+					(size 1.27 1.27)
+				)
+			)
+		)
 		(pin "1"
 		)
@@
 			)
 		)
+		(property "LCSC" "*"
+			(at 71.12 59.69 90)
+			(hide yes)
+			(show_name no)
+			(do_not_autoplace no)
+			(effects
+				(font
+					(size 1.27 1.27)
+				)
+			)
+		)
 		(pin "2"
 		)
@@
 			(hide yes)
 			(show_name no)
+			(do_not_autoplace no)
+			(effects
+				(font
+					(size 1.27 1.27)
+				)
+			)
+		)
+		(property "LCSC" "*"
+			(at 71.12 36.83 90)
+			(hide yes)
+			(show_name no)
