File: head/comms/wifi.kicad_sch (KiCad schematic)
At the start: 14 parts, among them U5 RTL8189FTV-VC-CG, Y3 26M

Commit message: finishing touches
Parts:
- AE1: LCSC (none) -> -
- C12, C14, C15, C16, C17, C18: value 0.1u -> 100n; LCSC (none) -> *
- C13: LCSC (none) -> *
- C26: LCSC (none) -> -; now left out of the parts list
- C57, C58: value 12p -> 10p; LCSC (none) -> *
- L2: LCSC (none) -> C2906877
Changed lines of the file:
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@@
 		(rev "1")
 		(company "team noon")
-		(comment 1 "NanoID: rI02tsXA")
+		(comment 1 "NanoID: GRG4UQ")
 		(comment 3 "github.com/team-noon/hw1")
 		(comment 4 "Drawn By: Sam")
@@
 			)
 		)
-		(property "Value" "0.1u"
+		(property "Value" "100n"
 			(at 60.96 52.07 90)
 			(hide yes)
@@
 		(property "Description" "Unpolarized capacitor"
 			(at 60.96 57.15 0)
+			(hide yes)
+			(show_name no)
+			(do_not_autoplace no)
+			(effects
+				(font
+					(size 1.27 1.27)
+				)
+			)
+		)
+		(property "LCSC" "*"
+			(at 60.96 57.15 90)
 			(hide yes)
 			(show_name no)
@@
 			)
 		)
+		(property "LCSC" "C2906877"
+			(at 144.78 82.55 90)
+			(hide yes)
+			(show_name no)
+			(do_not_autoplace no)
+			(effects
+				(font
+					(size 1.27 1.27)
+				)
+			)
+		)
 		(pin "1"
 		)
@@
 			)
 		)
-		(property "Value" "0.1u"
+		(property "Value" "100n"
 			(at 60.96 36.83 90)
 			(hide yes)
@@
 		(property "Description" "Unpolarized capacitor"
 			(at 60.96 41.91 0)
+			(hide yes)
+			(show_name no)
+			(do_not_autoplace no)
+			(effects
+				(font
+					(size 1.27 1.27)
+				)
+			)
+		)
+		(property "LCSC" "*"
+			(at 60.96 41.91 90)
 			(hide yes)
 			(show_name no)
@@
 			)
 		)
+		(property "LCSC" "-"
+			(at 157.48 82.55 90)
+			(hide yes)
+			(show_name no)
+			(do_not_autoplace no)
+			(effects
+				(font
+					(size 1.27 1.27)
+				)
+			)
+		)
 		(pin "2"
 		)
@@
 			)
 		)
-		(property "Value" "0.1u"
+		(property "Value" "100n"
 			(at 60.96 46.99 90)
 			(hide yes)
@@
 		(property "Description" "Unpolarized capacitor"
 			(at 60.96 52.07 0)
+			(hide yes)
+			(show_name no)
+			(do_not_autoplace no)
+			(effects
+				(font
+					(size 1.27 1.27)
+				)
+			)
+		)
+		(property "LCSC" "*"
+			(at 60.96 52.07 90)
 			(hide yes)
 			(show_name no)
@@
 			)
 		)
+		(property "LCSC" "*"
+			(at 60.96 67.31 90)
+			(hide yes)
+			(show_name no)
+			(do_not_autoplace no)
+			(effects
+				(font
+					(size 1.27 1.27)
+				)
+			)
+		)
 		(pin "1"
 		)
@@
 			)
 		)
-		(property "Value" "0.1u"
+		(property "Value" "100n"
 			(at 60.96 31.75 90)
 			(hide yes)
@@
 		(property "Description" "Unpolarized capacitor"
 			(at 60.96 36.83 0)
+			(hide yes)
+			(show_name no)
+			(do_not_autoplace no)
+			(effects
+				(font
+					(size 1.27 1.27)
+				)
+			)
+		)
+		(property "LCSC" "*"
+			(at 60.96 36.83 90)
 			(hide yes)
 			(show_name no)
@@
 			)
 		)
-		(property "Value" "0.1u"
+		(property "Value" "100n"
 			(at 60.96 57.15 90)
 			(hide yes)
@@
 		(property "Description" "Unpolarized capacitor"
 			(at 60.96 62.23 0)
+			(hide yes)
+			(show_name no)
+			(do_not_autoplace no)
+			(effects
+				(font
+					(size 1.27 1.27)
+				)
+			)
+		)
+		(property "LCSC" "*"
+			(at 60.96 62.23 90)
 			(hide yes)
 			(show_name no)
@@
 			)
 		)
-		(property "Value" "12p"
+		(property "Value" "10p"
 			(at 55.88 105.41 90)
 			(hide yes)
@@
 		(property "Description" "Unpolarized capacitor"
 			(at 55.88 110.49 0)
+			(hide yes)
+			(show_name no)
+			(do_not_autoplace no)
+			(effects
+				(font
+					(size 1.27 1.27)
+				)
+			)
+		)
+		(property "LCSC" "*"
+			(at 55.88 110.49 90)
 			(hide yes)
 			(show_name no)
@@
 			)
 		)
-		(property "Value" "12p"
+		(property "Value" "10p"
 			(at 55.88 97.79 90)
 			(hide yes)
@@
 		(property "Description" "Unpolarized capacitor"
 			(at 55.88 102.87 0)
+			(hide yes)
+			(show_name no)
+			(do_not_autoplace no)
+			(effects
+				(font
+					(size 1.27 1.27)
+				)
+			)
+		)
+		(property "LCSC" "*"
+			(at 55.88 102.87 90)
 			(hide yes)
 			(show_name no)
@@
 		(body_style 1)
 		(exclude_from_sim no)
-		(in_bom yes)
+		(in_bom no)
 		(on_board yes)
 		(in_pos_files yes)
@@
 		)
 		(property "Description" "Unpolarized capacitor"
+			(at 148.59 86.36 0)
+			(hide yes)
+			(show_name no)
+			(do_not_autoplace no)
+			(effects
+				(font
+					(size 1.27 1.27)
+				)
+			)
+		)
+		(property "LCSC" "-"
 			(at 148.59 86.36 0)
 			(hide yes)
@@
 			)
 		)
-		(property "Value" "0.1u"
+		(property "Value" "100n"
 			(at 60.96 41.91 90)
 			(hide yes)
@@
 			(hide yes)
 			(show_name no)
+			(do_not_autoplace no)
+			(effects
+				(font
+					(size 1.27 1.27)
+				)
+			)
+		)
+		(property "LCSC" "*"
+			(at 60.96 46.99 90)
+			(hide yes)
+			(show_name no)

Commit message: larger traces, swapped connector
Parts:
- AE1: now left out of the parts list
