File: motor/driver/motor-driver.kicad_pcb (KiCad board)
At the start: 2 copper layers, 36.4 x 35 mm, 62 parts, among them J1 DEBUG, J2 sensors, J3 controller, J4 motor, J5 thermal, J6 external, U2 LM66100DCK, U4 TJA1051TK-3, U5 RP114x, U6 MCT8316Z-Q1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

Commit message: implement driver
Parts:
- moved D7 0.30 mm to (55.5, 45.4)
Routing:
- net GND: track 177.3 -> 150.9 mm, vias 11 -> 12
- net Net-(D7-K): track 8.73 -> 11.4 mm
- net VBUS: track 24.6 -> 22.4 mm
- net Net-(U6-SW_BK): track 5.21 -> 4.49 mm
- net /DRVCC: track 13.1 -> 12.4 mm
- added copper zone on B.Cu, net Net-(D7-K)
- added copper zone on B.Cu, net Net-(F1-Pad1)
- added copper zone on B.Cu, net Net-(J3-Pin_5)
- added copper zone on F.Cu, net Net-(J3-Pin_5)
Other:
- board text added: "QLRRFD"
