File: motor/driver/motor-driver.kicad_pcb (KiCad board)
At the start: 2 copper layers, 36.4 x 35 mm, 62 parts, among them J1 DEBUG, J2 sensors, J3 controller, J4 motor, J5 thermal, J6 external, U2 LM66100DCK, U4 TJA1051TK-3, U5 RP114x, U6 MCT8316Z-Q1, U7 CH32L103F8U6

Commit message: driver rev 2
Parts:
- removed C9: 100n, Capacitor_SMD:C_0402_1005Metric
- removed D1: SZNUP2105L, Package_TO_SOT_SMD:SOT-23
- removed D10, D11, D6, D8, D9: PESD5V0L1UL, Diode_SMD:D_SOD-882
- removed R14: 1k, Resistor_SMD:R_0402_1005Metric
- removed TH1: Thermistor, Resistor_SMD:R_0402_1005Metric
- removed U4: TJA1051TK-3, Package_SON:HVSON-8-1EP_3x3mm_P0.65mm_EP1.6x2.4mm
- removed U6: MCT8316Z-Q1, misc:QFN-40_EP_5x7_Pitch0.5mm
- added C12: 1u, Capacitor_SMD:C_0402_1005Metric, F.Cu at (52.1, 63.6)
- added C20: 1u, Capacitor_SMD:C_0402_1005Metric, B.Cu at (42.0, 68.2)
- added C21: 2.2u, Capacitor_SMD:C_0402_1005Metric, B.Cu at (42.0, 73.2)
- added C22: 100n, Capacitor_SMD:C_0402_1005Metric, B.Cu at (60.0, 42.9)
- added C23: 100n, Capacitor_SMD:C_0402_1005Metric, B.Cu at (52.7, 42.4)
- added C24: 100n, Capacitor_SMD:C_0402_1005Metric, B.Cu at (48.7, 42.4)
- added C25: 2.2u, Capacitor_SMD:C_0402_1005Metric, F.Cu at (40.6, 46.1)
- added D3: SM712_SOT23, Package_TO_SOT_SMD:SOT-23, F.Cu at (52.5, 52.5)
- added R16: R_Small, Resistor_SMD:R_0402_1005Metric, B.Cu at (54.5, 47.2)
- added R17: R_Small, Resistor_SMD:R_0402_1005Metric, B.Cu at (54.0, 45.8)
- added R18: R_Small, Resistor_SMD:R_0402_1005Metric, B.Cu at (50.0, 45.8)
- added R19: R_Small, Resistor_SMD:R_0402_1005Metric, B.Cu at (50.5, 47.2)
- added U1: MCT8316Z, misc:QFN-40_EP_5x7_Pitch0.5mm, B.Cu at (50.5, 58.5)
- added U10: THVD1400D, Package_TO_SOT_SMD:SOT-583-8, B.Cu at (50.5, 43.5)
- added U3: TPS709, Package_TO_SOT_SMD:SOT-23-5, B.Cu at (42.5, 70.7)
- added U8: INA180A2, Package_TO_SOT_SMD:SOT-23-5, B.Cu at (62.5, 43.5)
- added U9: THVD1400D, Package_TO_SOT_SMD:SOT-583-8, B.Cu at (54.5, 43.5)
- C3: value 100n -> 2.2u
- C5: value 100n -> 2.2u; moved to B.Cu
- D5: value PESD5V0L1UL -> SM712_SOT23; footprint Diode_SMD:D_SOD-882 -> Package_TO_SOT_SMD:SOT-23; moved to F.Cu
- J3: value controller -> Conn_01x06_MountingPin; footprint Connector_Molex:Molex_Micro-Fit_3.0_43650-0512_1x05-1MP_P3.00mm_Horizontal -> Connector_Molex:Molex_Micro-Fit_3.0_43650-0600_1x06_P3.00mm_Horizontal
- R10, R11: moved to B.Cu
- R12: value 10k -> R_Small; moved to B.Cu
- R2: value 10 -> 100
- R3: value 10 -> R_Small
- R4: value 47k -> 100k; moved to B.Cu
- R5: value 10k -> 68k; moved to B.Cu
- R6: value 13.7k -> 5.1k
- R7: value 10k -> 5.1k
- R8: value 100 -> 4.7k
- moved C5 29.7 mm to (56.6, 73.2), turned to -90 degrees
- moved D5 23.7 mm to (46.5, 52.5), turned to -90 degrees
- moved C2 22.3 mm to (54.0, 63.5), turned to 90 degrees
- moved R8 19.0 mm to (41.7, 65.9)
- moved C4 14.1 mm to (58.5, 42.0)
- moved R12 12.6 mm to (51.0, 45.8)
- moved R7 11.6 mm to (53.0, 63.5), turned to 90 degrees
- moved U2 11.4 mm to (43.0, 56.5), turned to 180 degrees
- moved R6 10.5 mm to (52.0, 63.5), turned to 90 degrees
- moved C19 9.49 mm to (42.6, 54.9), turned to 0 degrees
- moved C8 9.38 mm to (44.5, 54.9), turned to 180 degrees
- moved C15 9.04 mm to (44.1, 58.8)
- moved J3 8.50 mm to (45.0, 49.1)
- moved R5 8.43 mm to (45.1, 58.8), turned to -90 degrees
- moved C6 8.24 mm to (42.6, 41.4), turned to 180 degrees
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Connections:
- net /CAN_RX renamed /SWDIO
- net /CAN_TX renamed /SWCLK
- C1 pad 1: /IN+ -> /Isense
- C1 pad 2: /IN- -> GND
- C12 pad 1: /DRVCC -> /AVDD
- C15 pad 1: Net-(U6-ILIM) -> Net-(U1MCT8316ZT-Q1-ILIM)
- C2 pad 1: VCC -> /VREF
- C3 pad 1: VDD -> VCC
- C4 pad 1: VDD -> VCC
- C5 pad 1: /Tb -> VCC
- C6 pad 1: /Tm -> /Tsense
- D5 pad 1: Net-(D5-K) -> /A2
- D5 pad 2: GND -> /B2
- J2 pad 1: /HPA -> /HPC
- J2 pad 3: /HPC -> /HPA
- J2 pad 5: /DRVCC -> /AVDD
- J3 pad 1: /CAN_H -> /B2
- J3 pad 2: /CAN_L -> /A2
- J3 pad 3: /ID -> /B1
- J3 pad 4: Net-(D7-K) -> /A1
- J3 pad 5: Net-(J3-Pin_5) -> Net-(D7-K)
- J4 pad 1: Net-(J4-Pin_1) -> /LC
- J4 pad 2: Net-(J4-Pin_2) -> /LB
- J4 pad 3: Net-(J4-Pin_3) -> /LA
- R1 pad 1: Net-(J3-Pin_5) -> Net-(J3-Pin_6)
- R10 pad 1: /DRVCC -> /AVDD
- R10 pad 2: /HNx -> /HPB
- R11 pad 1: /HNx -> /AVDD
- R11 pad 2: GND -> /HPC
- R12 pad 1: VCC -> Net-(U10-A)
- R12 pad 2: Net-(R12-Pad2) -> /A2
- R13 pad 1: /Tm -> /Tsense
- R2 pad 1: Net-(J3-Pin_5) -> Net-(R2-Pad1)
- R2 pad 2: /IN- -> /Isense
- R3 pad 1: GND -> Net-(U9-A)
- R3 pad 2: /IN+ -> /A1
- R4 pad 1: VBUS -> Net-(U1MCT8316ZT-Q1-ILIM)
- R4 pad 2: Net-(U6-~{SLEEP}) -> /AVDD
- R5 pad 1: Net-(U6-~{SLEEP}) -> Net-(U1MCT8316ZT-Q1-ILIM)
- R6 pad 1: /DRVCC -> /VREF
- R6 pad 2: Net-(U6-ILIM) -> /~{SLEEP}
- R7 pad 1: Net-(U6-ILIM) -> /VREF
- R7 pad 2: GND -> /~{FAULT}
- R8 pad 1: Net-(J5-Pin_2) -> /AVDD
- R8 pad 2: Net-(D5-K) -> /HPA
- U2 pad 3: GND -> VCCQ
- U2 pad 5: /SWST -> GND
- U7 pad 1: /IN+ -> /~{FAULT}
- U7 pad 10: /~{DRV_NSS} -> /DIR1
- U7 pad 11: /SCK -> /FGOUT
- U7 pad 12: /MISO -> /BRAKE
- U7 pad 13: /MOSI -> /DIR
- U7 pad 14: /LED -> /PWM
- U7 pad 15: /SWST -> /LED
- U7 pad 18: /CAN_S -> /EXT
- U7 pad 2: /IN- -> /Isense
- U7 pad 20: /Tb -> /~{SLEEP}
- U7 pad 3: /Tm -> /TX2
- U7 pad 4: /EXT -> /RX2
- U7 pad 5: /ID -> /DIR2
- U7 pad 6: /DRVOFF -> /Tsense
- U7 pad 7: /~{FAULT} -> /DRVOFF
- U7 pad 8: /FGOUT -> /TX1
- U7 pad 9: /PWM -> /RX1
Routing:
- net /Tsense: track 0.00 -> 37.1 mm, vias 0 -> 3
- net /Tm: track 30.2 -> 0.00 mm, vias 2 -> 0
- net /VREF: track 0.00 -> 28.8 mm, vias 0 -> 2
- net /~{SLEEP}: track 0.00 -> 27.7 mm, vias 0 -> 2
- net /AVDD: track 0.00 -> 26.9 mm, vias 0 -> 1
- net /IN+: track 24.0 -> 0.00 mm
- net /DIR: track 0.00 -> 19.9 mm
- net /Isense: track 0.00 -> 19.6 mm
- net VBUS: track 22.4 -> 41.8 mm, vias 3 -> 4
- net VDD: track 27.7 -> 9.16 mm, vias 2 -> 0
- net /IN-: track 17.6 -> 0.00 mm
- net /~{FAULT}: track 11.6 -> 28.4 mm
- net VCC: track 87.2 -> 70.5 mm, vias 4 -> 8
- net /DIR1: track 0.00 -> 16.4 mm, vias 0 -> 2
- net /TX1: track 0.00 -> 14.5 mm, vias 0 -> 2
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- added copper zone on B.Cu, net /LA
- added copper zone on B.Cu, net /LB
- added copper zone on B.Cu, net /LC
- added copper zone on B.Cu, net Net-(J3-Pin_6)
- added copper zone on F.Cu, net VBUS
- removed copper zone on B.Cu, net Net-(J3-Pin_5)
- removed copper zone on F.Cu, net Net-(J3-Pin_5)
- removed copper zone on B.Cu, net Net-(J4-Pin_1)
- removed copper zone on B.Cu, net Net-(J4-Pin_2)
- removed copper zone on B.Cu, net Net-(J4-Pin_3)
Other:
- board text added: "X2AJPD"
- board text removed: "QLRRFD"

Commit message: motor/driver - final touches
Parts:
- removed C25: 2.2u, Capacitor_SMD:C_0402_1005Metric
- C1, C14, C15, C2, C22, C23, C24, C6: value 100n -> 100n (16V)
- C10: value 47n -> 47n (50V)
- C11, C20: value 1u -> 1u (50V)
- C12, C7, C8: value 1u -> 1u (16V)
- C13: value 22u -> 22u (16V)
- C16: value 100n -> 100n(50V)
- C17: value 10u / HV -> 10u (50V)
- C18: value 100u / HV -> 100u (50V)
- C19: value 10u -> 10u (10V)
- C21, C4, C5: value 2.2u -> 2.2u (16V)
- C3: value 2.2u -> 2.2u (16V); moved to F.Cu
- D2: moved to B.Cu
- H1, H2, H3, H4: value MountingHole_Pad -> MountingScrew
- J3: value Conn_01x06_MountingPin -> master bus
- J6: value external -> satellite
- R12, R17, R18, R3: value R_Small -> 10
- R16, R19: value R_Small -> 120
- moved D2 21.7 mm to (46.8, 73.4)
- moved C3 6.59 mm to (40.7, 46.3), turned to -90 degrees
- moved C13 3.90 mm to (47.8, 51.0), turned to 0 degrees
- moved C6 3.68 mm to (46.1, 42.5), turned to 45 degrees
- moved C19 2.17 mm to (44.1, 56.5), turned to -90 degrees
- moved C7 1.67 mm to (44.9, 53.2), turned to 180 degrees
- moved C8 1.26 mm to (43.5, 54.1), turned to 90 degrees
- moved C23 1.24 mm to (53.0, 41.2), turned to 180 degrees
- moved U5 1.08 mm to (44.9, 54.5), turned to 0 degrees
- moved C1 0.87 mm to (43.8, 41.0), turned to 180 degrees
- moved R12 0.71 mm to (51.5, 45.3)
- moved R18 0.71 mm to (50.5, 45.3)
- moved R19 0.71 mm to (51.0, 46.7)
- moved U10 0.71 mm to (51.0, 43.0)
- moved R16 0.58 mm to (54.2, 46.7)
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Connections:
- C14 pad 1: VCCQ -> VCC
- C19 pad 1: VCCQ -> VCC
- D2 pad 1: VCCQ -> VCC
- J1 pad 1: VCCQ -> Net-(J1-Pin_1)
- U2 pad 1: VCC -> Net-(J1-Pin_1)
- U2 pad 3: VCCQ -> VCC
- U2 pad 6: VCCQ -> VCC
- U7 pad 19: VCCQ -> VCC
Routing:
- net VCCQ: track 28.2 -> 0.00 mm, vias 3 -> 0
- net /LED: track 8.64 -> 35.1 mm, vias 1 -> 2
- net GND: track 161.3 -> 181.3 mm, vias 29 -> 24
- net VCC: track 70.5 -> 87.1 mm
- net Net-(J1-Pin_1): track 0.00 -> 2.73 mm, vias 0 -> 1
- net /Tsense: track 37.1 -> 34.9 mm, vias 3 -> 2
- net Net-(J3-Pin_6): track 5.08 -> 7.03 mm
- net /DIR1: track 16.4 -> 14.5 mm
- net /B2: track 8.63 -> 10.2 mm
- net /A2: track 6.65 -> 8.14 mm
- net /DIR2: track 8.01 -> 9.39 mm, vias 2 -> 0
- net /RX1: track 14.2 -> 12.9 mm
- net /A1: track 5.17 -> 6.38 mm
- net /Isense: track 19.6 -> 20.8 mm
- net /EXT: track 38.8 -> 39.7 mm
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