File: motor/servo/motor-servo.kicad_pcb (KiCad board)
At the start: 2 copper layers, 36.4 x 35 mm, 50 parts, among them J1 DEBUG, J2 servo, J3 Conn_01x06_MountingPin, J6 satellite, U1 SY8205, U10 THVD1400D, U2 LM66100DCK, U5 RP114x, U7 CH32L103F8U6, U8 INA180A2, U9 THVD1400D

Commit message: changed buck
Parts:
- removed C2: 100n, Capacitor_SMD:C_0402_1005Metric
- removed C3: 1u, Capacitor_SMD:C_0402_1005Metric
- removed C4: C_Small, Capacitor_SMD:C_0402_1005Metric
- removed C5: 100p, Capacitor_SMD:C_0402_1005Metric
- removed C9: 10u, Capacitor_SMD:C_0805_2012Metric
- removed L1: 4.2u, Inductor_SMD:L_Wuerth_HCM-1190
- removed R4: 100k, Resistor_SMD:R_0402_1005Metric
- removed R5: 13k, Resistor_SMD:R_0402_1005Metric
- removed U1: SY8205, Package_SO:Infineon_PG-DSO-8-43
- added C12: 10u (HV), Capacitor_SMD:C_0805_2012Metric, F.Cu at (62.7, 58.1)
- added C15: 1u (HV), Capacitor_SMD:C_0603_1608Metric, F.Cu at (62.5, 56.3)
- added C16: 100n, Capacitor_SMD:C_0402_1005Metric, F.Cu at (60.7, 54.4)
- added C17: 2.2u, Capacitor_SMD:C_0402_1005Metric, F.Cu at (59.7, 54.4)
- added C18: 22p, Capacitor_SMD:C_0402_1005Metric, F.Cu at (56.3, 53.3)
- added L2: 2u, misc:0630CDMCD_DS, F.Cu at (52.5, 57.5)
- added R11: 150k, Resistor_SMD:R_0402_1005Metric, F.Cu at (58.3, 53.8)
- added R13: 100k, Resistor_SMD:R_0402_1005Metric, F.Cu at (56.3, 52.3)
- added R15: 13k, Resistor_SMD:R_0402_1005Metric, F.Cu at (58.3, 54.8)
- added U3: SY8366H, misc:QFN3x3-12, F.Cu at (59.0, 57.3)
- moved F1 0.60 mm to (62.9, 52.9)
Connections:
- U7 pad 7: unconnected-(U7-PA7-Pad7) -> /PG
Routing:
- net /PG: track 0.00 -> 20.3 mm, vias 0 -> 3
- net GND: track 84.7 -> 100.9 mm, vias 12 -> 21
- net Net-(U1-LX): track 13.7 -> 0.00 mm
- net Net-(U3-LX): track 0.00 -> 9.20 mm, vias 0 -> 2
- net Net-(U3-FB): track 0.00 -> 4.85 mm
- net Net-(F1-Pad1): track 3.44 -> 0.00 mm
- net Net-(U1-FB): track 3.36 -> 0.00 mm
- net VBUS: track 16.7 -> 14.4 mm, vias 0 -> 2
- net Net-(U1-VCC): track 1.39 -> 0.00 mm
- net Net-(U1-SS): track 1.38 -> 0.00 mm
- net Net-(U1-BS): track 1.38 -> 0.00 mm
- net Net-(C18-Pad2): track 0.00 -> 1.22 mm
- net Net-(U3-BS): track 0.00 -> 1.21 mm
- net VDD: track 25.2 -> 24.1 mm, vias 1 -> 0
- net Net-(U3-VCC): track 0.00 -> 0.99 mm
- added copper zone on F.Cu, net Net-(U3-LX)

Commit message: motor/servo - final touches
Parts:
- removed C25: 2.2u, Capacitor_SMD:C_0402_1005Metric
- C1, C14, C16, C22, C23, C24: value 100n -> 100n (16V)
- C10, C6: value 22u -> 22u (16V); footprint Capacitor_SMD:C_0805_2012Metric -> Capacitor_SMD:C_0603_1608Metric
- C11: value 220u -> 220u (16V)
- C12: value 10u (HV) -> 10u (50V); footprint Capacitor_SMD:C_0805_2012Metric -> Capacitor_SMD:C_0603_1608Metric
- C15: value 1u (HV) -> 1u (50V); footprint Capacitor_SMD:C_0603_1608Metric -> Capacitor_SMD:C_0402_1005Metric
- C17: value 2.2u -> 2.2u (16V)
- C18: value 22p -> 22p (16V)
- C19: value 10u -> 10u (16V)
- C7, C8: value 1u -> 1u (16V)
- D2: moved to B.Cu
- D3, D5: moved to F.Cu
- H1, H2, H3, H4: value MountingHole_Pad -> MountingScrew
- J3: value Conn_01x06_MountingPin -> master bus
- R12, R17, R18, R3: value R_Small -> 10
- R16, R19: value R_Small -> 120
- moved D2 21.7 mm to (46.8, 73.4)
- moved C23 5.00 mm to (57.7, 42.4), turned to 0 degrees
- moved C19 4.44 mm to (47.0, 59.9), turned to 180 degrees
- moved C8 4.36 mm to (49.4, 60.0)
- moved C7 1.73 mm to (49.4, 57.4), turned to 180 degrees
- moved U5 1.70 mm to (49.4, 58.7), turned to 0 degrees
- moved C15 1.40 mm to (62.4, 57.7)
- moved U2 1.27 mm to (47.0, 58.3), turned to 0 degrees
- moved C16 1.00 mm to (60.7, 55.4)
- moved C17 1.00 mm to (59.7, 55.4)
- moved C18 1.00 mm to (56.3, 54.3)
- moved L2 1.00 mm to (52.5, 58.5)
- moved R11 1.00 mm to (58.3, 54.8)
- moved R13 1.00 mm to (56.3, 53.3)
- moved R15 1.00 mm to (58.3, 55.8)
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Connections:
- C14 pad 1: VCCQ -> VCC
- C19 pad 1: VCCQ -> VCC
- D2 pad 1: VCCQ -> VCC
- D3 pad 1: /B1 -> /A1
- D3 pad 2: /A1 -> /B1
- D5 pad 1: /B2 -> /A2
- D5 pad 2: /A2 -> /B2
- J1 pad 1: VCCQ -> Net-(J1-Pin_1)
- U2 pad 1: VCC -> Net-(J1-Pin_1)
- U2 pad 3: VCCQ -> VCC
- U2 pad 6: VCCQ -> VCC
- U7 pad 19: VCCQ -> VCC
Routing:
- net VCCQ: track 32.1 -> 0.00 mm, vias 3 -> 0
- net /LED: track 8.64 -> 32.4 mm, vias 1 -> 0
- net GND: track 100.9 -> 82.6 mm, vias 21 -> 17
- net VCC: track 73.1 -> 87.2 mm, vias 5 -> 8
- net /PG: track 20.3 -> 24.0 mm
- net VDD: track 24.1 -> 27.3 mm, vias 0 -> 1
- net Net-(F1-Pad1): track 0.00 -> 2.84 mm
- net Net-(J1-Pin_1): track 0.00 -> 2.16 mm, vias 0 -> 1
- net /DIR1: track 16.6 -> 14.5 mm
- net /RX1: track 14.1 -> 12.7 mm
- net /EXT: track 44.2 -> 45.3 mm
- net /DIR2: track 8.01 -> 8.85 mm, vias 2 -> 0
- net /A2: track 7.43 -> 8.13 mm
- net /B2: track 9.41 -> 10.1 mm
- net /servo: track 49.6 -> 50.3 mm
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