File: motor/servo/motor-servo.kicad_sch (KiCad schematic)
At the start: 50 parts, among them J1 DEBUG, J2 servo, J3 Conn_01x06_MountingPin, J6 satellite, U1 SY8205, U10 THVD1400D, U2 LM66100DCK, U5 RP114x, U7 CH32L103F8U6, U8 INA180A2, U9 THVD1400D

Commit message: changed buck
Parts:
- removed C2: 100n, Capacitor_SMD:C_0402_1005Metric, symbol Device:C_Small
- removed C3: 1u, Capacitor_SMD:C_0402_1005Metric, symbol Device:C_Small
- removed C4: C_Small, Capacitor_SMD:C_0402_1005Metric, symbol Device:C_Small
- removed C5: 100p, Capacitor_SMD:C_0402_1005Metric, symbol Device:C_Small
- removed C9: 10u, Capacitor_SMD:C_0805_2012Metric, symbol Device:C
- removed L1: 4.2u, Inductor_SMD:L_Wuerth_HCM-1190, symbol Device:L
- removed R4: 100k, Resistor_SMD:R_0402_1005Metric, symbol Device:R_Small
- removed R5: 13k, Resistor_SMD:R_0402_1005Metric, symbol Device:R_Small
- removed U1: SY8205, Package_SO:Infineon_PG-DSO-8-43, symbol silergy:SY8205
- added C12: 10u (HV), Capacitor_SMD:C_0805_2012Metric, symbol Device:C
- added C15: 1u (HV), Capacitor_SMD:C_0603_1608Metric, symbol Device:C
- added C16: 100n, Capacitor_SMD:C_0402_1005Metric, symbol Device:C
- added C17: 2.2u, Capacitor_SMD:C_0402_1005Metric, symbol Device:C
- added C18: 22p, Capacitor_SMD:C_0402_1005Metric, symbol Device:C_Small
- added L2: 2u, misc:0630CDMCD_DS, symbol Device:L
- added R11: 150k, Resistor_SMD:R_0402_1005Metric, symbol Device:R_Small
- added R13: 100k, Resistor_SMD:R_0402_1005Metric, symbol Device:R
- added R15: 13k, Resistor_SMD:R_0402_1005Metric, symbol Device:R
- added U3: SY8366H, misc:QFN3x3-12, symbol silergy:SY8366H
Connections:
- net GND: now also C12.2, C15.2, C17.2, R15.1, U3.1 (GND), U3.10 (ILIM)
- net VDD: now also C18.1, L2.2, R13.1
- net PG: now reaches U7.7 (PA7)
- net PG: now also U3.11 (PG)
- net VBUS renamed IN
- net IN: now also C12.1, C15.1, U3.12 (EN), U3.5 (IN), U3.6 (IN)
- new net: C17.1, U3.8 (VCC)
- new net: R11.2, R13.2, R15.2, U3.9 (FB)
- new net: C16.2, L2.1, U3.2 (LX)
- new net: C16.1, U3.7 (BS)
- new net: C18.2, R11.1
- no-connect marks 1 -> 7
Other:
- note added: "6A max"

Commit message: motor/servo - final touches
Parts:
- removed C25: 2.2u, Capacitor_SMD:C_0402_1005Metric, symbol Device:C
- removed H1, H2, H3, H4: MountingHole_Pad, MountingHole:MountingHole_2.2mm_M2_DIN965_Pad, symbol Mechanical:MountingHole_Pad
- added H1, H2, H3, H4: MountingScrew, MountingHole:MountingHole_2.2mm_M2_DIN965_Pad, symbol Auxiliary_Items:MountingScrew
- C1: value 100n -> 100n (16V); footprint (none) -> Capacitor_SMD:C_0402_1005Metric; LCSC (none) -> *
- C10, C6: value 22u -> 22u (16V); footprint Capacitor_SMD:C_0805_2012Metric -> Capacitor_SMD:C_0603_1608Metric; LCSC C98190 -> C2762594
- C11: value 220u -> 220u (16V)
- C12: value 10u (HV) -> 10u (50V); footprint Capacitor_SMD:C_0805_2012Metric -> Capacitor_SMD:C_0603_1608Metric; LCSC (none) -> (C194427)
- C14: value 100n -> 100n (16V); LCSC C77020 -> *
- C15: value 1u (HV) -> 1u (50V); footprint Capacitor_SMD:C_0603_1608Metric -> Capacitor_SMD:C_0402_1005Metric; LCSC C307331 -> *
- C16: value 100n -> 100n (16V); LCSC C60474 -> *
- C17: value 2.2u -> 2.2u (16V); LCSC C12530 -> *
- C18: value 22p -> 22p (16V); LCSC C106203 -> *
- C19: value 10u -> 10u (16V); LCSC C315248 -> *
- C22, C23, C24: value 100n -> 100n (16V); LCSC (none) -> *
- C7, C8: value 1u -> 1u (16V); LCSC C7001784 -> *
- J3: value Conn_01x06_MountingPin -> master bus
- R11, R13, R15: LCSC (none) -> *
- R12, R17, R18, R3: value R_Small -> 10; LCSC (none) -> *
- R16, R19: value R_Small -> 120; LCSC (none) -> *; now not fitted
- R2: footprint (none) -> Resistor_SMD:R_0402_1005Metric; LCSC (none) -> *
- U5: LCSC C194610 -> C246258
Connections:
- net A1: now also D3.1 (A1); no longer D3.2 (A2)
- net A2: now also D5.1 (A1); no longer D5.2 (A2)
- net B1: now also D3.2 (A2); no longer D3.1 (A1)
- net B2: now also D5.2 (A2); no longer D5.1 (A1)
- net GND: now also H1.1 (PAD), H2.1 (PAD), H3.1 (PAD), H4.1 (PAD)
- net VCC: now also C14.1, C19.1, D2.1 (VDD), U2.3 (~{CE}), U2.6 (VOUT), U7.19 (VDD); no longer U2.1 (VIN)
- removed net VCCQ: C14.1, C19.1, D2.1 (VDD), J1.1 (Pin_1), U2.3 (~{CE}), U2.6 (VOUT), U7.19 (VDD)
- new net: J1.1 (Pin_1), U2.1 (VIN)
Other:
- moved on the sheet: C14
