File: motor/satellite/motor-satellite.kicad_pcb (KiCad board)
At the start: 2 copper layers, 10 x 10 mm, 9 parts, among them J3 Conn_01x04_MountingPin, J6 Conn_01x03_MountingPin, U1 CH32V005D6U6, U3 SC4251

Commit message: motor/satellite - final touches
Parts:
- added H1: MountingScrew, MountingHole:MountingHole_2.2mm_M2_Pad, F.Cu at (50.0, 45.0)
- added H2: MountingScrew, MountingHole:MountingHole_2.2mm_M2_Pad, F.Cu at (40.0, 45.0)
- moved D2 7.15 mm to (42.2, 48.6), turned to 0 degrees
- moved C3 0.60 mm to (46.1, 43.4), turned to 0 degrees
Routing:
- net /LED: track 10.8 -> 1.42 mm
- net GND: track 13.0 -> 18.1 mm, vias 5 -> 4
- net /TX: track 6.75 -> 4.69 mm
Other:
- board size 10 x 10 mm -> 15 x 10 mm
