File: motor/satellite/motor-satellite.kicad_sch (KiCad schematic)
At the start: 9 parts, among them J3 Conn_01x04_MountingPin, J6 Conn_01x03_MountingPin, U1 CH32V005D6U6, U3 SC4251

Commit message: motor/satellite - final touches
Parts:
- added H1, H2: MountingScrew, MountingHole:MountingHole_2.2mm_M2_Pad, symbol Auxiliary_Items:MountingScrew
- C1, C2, C3: LCSC (none) -> *
- TP1: LCSC (none) -> -
- U1: LCSC (none) -> C49006243
Connections:
- net GND: now also H1.1 (PAD), H2.1 (PAD)
